File: kiku.kicad_sch (KiCad schematic)
At the start: 0 parts

Commit message: add the microcontroller and stuff
Parts:
- added J1: USB_C_Receptacle_USB2.0_16P, symbol Connector:USB_C_Receptacle_USB2.0_16P
- added U1: ESP32-S3-WROOM-1, RF_Module:ESP32-S3-WROOM-1, symbol RF_Module:ESP32-S3-WROOM-1
- added U2: Value, libraries:Wio-SX1262 PCB Package, symbol Wio-SX1262 Schematic Package:MODULE-WIO-SX1262
Connections:
- new net: U1.1 (GND), U1.40 (GND), U1.41 (GND)
- new net: J1.A1 (GND), J1.A12 (GND), J1.B1 (GND), J1.B12 (GND)
- new net: J1.A4 (VBUS), J1.A9 (VBUS), J1.B4 (VBUS), J1.B9 (VBUS)
- new net D+: J1.A6 (D+), J1.B6 (D+), U1.14 (USB_D+)
- new net D-: J1.A7 (D-), J1.B7 (D-), U1.13 (USB_D-)

Commit message: a lot of connections are done
Parts:
- U2: value Value -> Wio-sx1262-n
Connections:
- net GND: now reaches U1.1 (GND), U1.40 (GND), U1.41 (GND)
- net GND: now also J1.A1 (GND), J1.A12 (GND), J1.B1 (GND), J1.B12 (GND), U2.10 (GND2), U2.7 (GND1)
- net +3.3V: now reaches U1.2 (3V3)
- net +3.3V: now also J1.A4 (VBUS), J1.A9 (VBUS), J1.B4 (VBUS), J1.B9 (VBUS)
Other:
- moved on the sheet: U1

Commit message: quite a bit of changes, still not finished with the schematic. havent committed in a while
Parts:
- removed J1: USB_C_Receptacle_USB2.0_16P, symbol Connector:USB_C_Receptacle_USB2.0_16P
- added C3, C4, C5, C6, C7, C8: 1 µF, Capacitor_SMD:C_0603_1608Metric, symbol Device:C
- added C9: 10 µF, Capacitor_SMD:C_0603_1608Metric, symbol Device:C
- added J1: BM02B-SRSS-TB LFSN, libraries:CONN_BM02B-SRSS-TB_JST, symbol libraries:BM02B-SRSS-TB_LFSN
- added J2: USB_C_Receptacle_USB2.0_16P, Connector_USB:USB_C_Receptacle_GCT_USB4105-xx-A_16P_TopMnt_Horizontal, symbol Connector:USB_C_Receptacle_USB2.0_16P
- added J3: Conn_Coaxial, Connector_Coaxial:SMA_Molex_73251-1153_EdgeMount_Horizontal, symbol Connector:Conn_Coaxial
- added R10: 2.4 kΩ, Resistor_SMD:R_0402_1005Metric, symbol Device:R
- added R4, R5: 5.1k, Resistor_SMD:R_0402_1005Metric, symbol Device:R
- added R6, R7: 10 kΩ, Resistor_SMD:R_0402_1005Metric, symbol Device:R
- added R8: 390 kΩ, Resistor_SMD:R_0402_1005Metric, symbol Device:R
- added R9: 100 kΩ, Resistor_SMD:R_0402_1005Metric, symbol Device:R
- added SW1, SW2: SW_SPST, Button_Switch_SMD:SW_SPST_B3U-1100P, symbol Switch:SW_SPST
- added TP1, TP2: TestPoint, TestPoint:TestPoint_Keystone_5010-5014_Multipurpose, symbol Connector:TestPoint
- added U4: AMS1117-3.3, Package_TO_SOT_SMD:SOT-223-3_TabPin2, symbol Regulator_Linear:AMS1117-3.3
- added U6: BQ25185DLHR, libraries:WSON10_DLH_TEX, symbol libraries:BQ25185DLHR
Connections:
- net +3.3V: now also U2.8 (VCC)
- net D+: now also J2.A7 (D-), J2.B7 (D-)
- net D-: now also J2.A6 (D+), J2.B6 (D+)
- net GND: now also C3.2, C4.2, C5.2, C6.2, C7.1, C8.1, C9.2, J1.2, J2.A1 (GND), J2.A12 (GND), J2.B1 (GND), J2.B12 (GND), J3.2 (Ext), R10.1, R4.2, R5.2, R9.2, SW1.1 (A), SW2.1 (A), U4.1 (GND), U6.5 (GND)
- net RESET: now reaches U1.12 (IO8)
- net RESET: now also U2.5 (RST)
- net MISO: now reaches U1.15 (IO3)
- net MISO: now also U2.2 (MISO)
- net BOOT: now reaches U1.27 (IO0)
- net BOOT: now also C6.1, R7.2, SW1.2 (B)
- net en: now reaches U1.3 (EN)
- net en: now also C5.1, R6.2, SW2.2 (B)
- net BattVoltage: now reaches U1.39 (IO1)
- net BattVoltage: now also R8.2, R9.1
- net SCK: now reaches U1.5 (IO5)
- net SCK: now also U2.4 (SCK)
- net MOSI: now reaches U1.6 (IO6)
- net MOSI: now also U2.3 (MOSI)
- net BUSY: now reaches U1.8 (IO15)
- net BUSY: now also U2.11 (BUSY)
- net DIO1: now reaches U1.9 (IO16)
- net DIO1: now also U2.12 (DIO1)
- net NSS: now reaches U2.6 (NSS)
- net ANT: now reaches U2.9 (ANT)
- net ANT: now also J3.1 (In)
- new net: J2.A5 (CC1), R4.1
- new net: R10.2, U6.7 (ILIM/VSET)
- new net: J2.B5 (CC2), R5.1
- new net +3V3: C3.1, R6.1, R7.1, U4.2 (VO)
- new net +4.5V: C4.1, C9.1, U4.3 (VI), U6.1 (SYS)
- new net +BATT: C8.2, J1.1, R8.1, U6.2 (BAT)
- new net VBUS: C7.2, J2.A4 (VBUS), J2.A9 (VBUS), J2.B4 (VBUS), J2.B9 (VBUS), TP1.1, U6.10 (IN)
- no-connect marks 0 -> 3
Other:
- note added: "LoRa Module"
- note added: "Microcontroller"
- note added: "SMA connector"
- note added: "Switches + voltage"
- note added: "battery connector,charging and voltage regulator"
- note added: "usb-c"
- moved on the sheet: U1, U2

Commit message: more work on the power stuff
Parts:
- added R11: 300Ω, Resistor_SMD:R_0402_1005Metric, symbol Device:R
- added SW3: RESET CHARGER, Button_Switch_SMD:SW_SPST_B3U-1100P, symbol Switch:SW_SPST
- SW1: value SW_SPST -> BOOT
- SW2: value SW_SPST -> EN
Connections:
- net GND: now also R11.1, SW3.2 (B)
- net at U6.6 (TS/MR): now also SW3.1 (A)
- net at U6.8 (ISET): now also R11.2
Other:
- moved on the sheet: C8

Commit message: mostly finished on the schematic, possibly starting on the routing
Parts:
- added R12: 10 kΩ, Resistor_SMD:R_0402_1005Metric, symbol Device:R
Connections:
- net VBUS: now also R12.1
- net CHGSWITCH: now reaches U1.38 (IO2)
- net CHGSWITCH: now also U6.4 (/CE), R12.2
- net BattVoltage renamed BATTVOLT
Changed lines of the file:
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@@
 	(wire
 		(pts
+			(xy 34.29 154.94) (xy 46.99 154.94)
+		)
+		(stroke
+			(width 0)
+			(type default)
+		)
+	)
+	(wire
+		(pts
 			(xy 93.98 36.83) (xy 93.98 39.37)
 		)
@@
 	(wire
 		(pts
+			(xy 34.29 149.86) (xy 34.29 154.94)
+		)
+		(stroke
+			(width 0)
+			(type default)
+		)
+	)
+	(wire
+		(pts
 			(xy 121.92 63.5) (xy 118.11 63.5)
 		)
@@
 		)
 	)
+	(global_label "CHGSWITCH"
+		(shape input)
+		(at 46.99 154.94 0)
+		(fields_autoplaced yes)
+		(effects
+			(font
+				(size 1.27 1.27)
+			)
+			(justify left)
+		)
+		(property "Intersheetrefs" "${INTERSHEET_REFS}"
+			(at 60.6795 154.94 0)
+			(hide yes)
+			(show_name no)
+			(do_not_autoplace no)
+			(effects
+				(font
+					(size 1.27 1.27)
+				)
+				(justify left)
+			)
+		)
+	)
 	(global_label "BOOT"
 		(shape input)
@@
 		)
 	)
-	(global_label "BattVoltage"
+	(global_label "BATTVOLT"
 		(shape input)
 		(at 176.53 44.45 0)
@@
 		)
 		(property "Intersheetrefs" "${INTERSHEET_REFS}"
-			(at 190.4007 44.45 0)
+			(at 188.2238 44.45 0)
 			(hide yes)
 			(show_name no)
@@
 		)
 	)
+	(global_label "CHGSWITCH"
+		(shape input)
+		(at 176.53 46.99 0)
+		(fields_autoplaced yes)
+		(effects
+			(font
+				(size 1.27 1.27)
+			)
+			(justify left)
+		)
+		(property "Intersheetrefs" "${INTERSHEET_REFS}"
+			(at 190.2195 46.99 0)
+			(hide yes)
+			(show_name no)
+			(do_not_autoplace no)
+			(effects
+				(font
+					(size 1.27 1.27)
+				)
+				(justify left)
+			)
+		)
+	)
 	(global_label "MOSI"
 		(shape input)
@@
 		)
 	)
-	(global_label "BattVoltage"
+	(global_label "BATTVOLT"
 		(shape input)
 		(at 105.41 63.5 90)
@@
 		)
 		(property "Intersheetrefs" "${INTERSHEET_REFS}"
-			(at 105.41 49.6293 90)
+			(at 105.41 51.8062 90)
 			(hide yes)
 			(show_name no)
@@
 	)
 	(symbol
+		(lib_id "power:VBUS")
+		(at 46.99 147.32 0)
+		(unit 1)
+		(body_style 1)
+		(exclude_from_sim no)
+		(in_bom yes)
+		(on_board yes)
+		(in_pos_files yes)
+		(dnp no)
+		(fields_autoplaced yes)
+		(property "Reference" "#PWR033"
+			(at 46.99 151.13 0)
+			(hide yes)
+			(show_name no)
+			(do_not_autoplace no)
+			(effects
+				(font
+					(size 1.27 1.27)
+				)
+			)
+		)
+		(property "Value" "VBUS"
+			(at 46.99 142.24 0)
+			(show_name no)
+			(do_not_autoplace no)
+			(effects
+				(font
+					(size 1.27 1.27)
+				)
+			)
+		)
+		(property "Footprint" ""
+			(at 46.99 147.32 0)
+			(hide yes)
+			(show_name no)
+			(do_not_autoplace no)
+			(effects
+				(font
+					(size 1.27 1.27)
+				)
+			)
+		)
+		(property "Datasheet" ""
+			(at 46.99 147.32 0)
+			(hide yes)
+			(show_name no)
+			(do_not_autoplace no)
+			(effects
+				(font
+					(size 1.27 1.27)
+				)
+			)
+		)
+		(property "Description" "Power symbol creates a global label with name \"VBUS\""
+			(at 46.99 147.32 0)
+			(hide yes)
+			(show_name no)
+			(do_not_autoplace no)
+			(effects
+				(font
+					(size 1.27 1.27)
+				)
+			)
+		)
+		(pin "1"
+		)
+		(instances
+			(project "kiku"
+				(path "/da0f8494-32d1-465d-8e52-ef98de02d741"
+					(reference "#PWR033")
+					(unit 1)
+				)
+			)
+		)
+	)
+	(symbol
 		(lib_id "power:GND")
 		(at 119.38 49.53 0)
@@
 					(unit 1)
 				)
+			)
+		)
+	)
+	(symbol
+		(lib_id "Device:R")
+		(at 46.99 151.13 0)
+		(unit 1)
+		(body_style 1)
+		(exclude_from_sim no)
+		(in_bom yes)
+		(on_board yes)
+		(in_pos_files yes)
+		(dnp no)
+		(fields_autoplaced yes)
+		(property "Reference" "R12"
+			(at 49.53 149.8599 0)
+			(show_name no)
+			(do_not_autoplace no)
+			(effects
+				(font
+					(size 1.27 1.27)
+				)
+				(justify left)
+			)
+		)
+		(property "Value" "10 kΩ"
+			(at 49.53 152.3999 0)
+			(show_name no)
+			(do_not_autoplace no)
+			(effects
+				(font
+					(size 1.27 1.27)
+				)
+				(justify left)
+			)
+		)
+		(property "Footprint" "Resistor_SMD:R_0402_1005Metric"
+			(at 45.212 151.13 90)
+			(hide yes)
+			(show_name no)
+			(do_not_autoplace no)
+			(effects
+				(font
+					(size 1.27 1.27)
+				)
+			)
+		)
+		(property "Datasheet" ""
+			(at 46.99 151.13 0)
+			(hide yes)
+			(show_name no)
+			(do_not_autoplace no)
+			(effects
+				(font
+					(size 1.27 1.27)
+				)
+			)
+		)
+		(property "Description" "Resistor"
+			(at 46.99 151.13 0)
+			(hide yes)
+			(show_name no)
+			(do_not_autoplace no)
+			(effects
+				(font
+					(size 1.27 1.27)
+				)
+			)
+		)
+		(pin "2"
+		)
+		(pin "1"
+		)
+		(instances
+			(project "kiku"
+				(path "/da0f8494-32d1-465d-8e52-ef98de02d741"
+					(reference "R12")
+					(unit 1)
+				)

Commit message: think im mostly finished
Parts:
- added C10, C11: 1 µF, Capacitor_SMD:C_0603_1608Metric, symbol Device:C
- added R13: 10 kΩ, Resistor_SMD:R_0402_1005Metric, symbol Device:R
- added U5: AMS1117-3.3, Package_TO_SOT_SMD:SOT-223-3_TabPin2, symbol Regulator_Linear:AMS1117-3.3
- TP1: value TestPoint -> PWR
- TP2: value TestPoint -> GND
Connections:
- net +3.3V: now also C3.1, U4.2 (VO), R13.1
- net +3V3: no longer C3.1, U4.2 (VO)
- net BUSY: now also U1.5 (IO5); no longer U1.8 (IO15)
- net GND: now also TP2.1, C10.2, C11.2, U5.1 (GND)
- net MOSI: now also U1.12 (IO8); no longer U1.6 (IO6)
- net RESET: now also U1.6 (IO6); no longer U1.12 (IO8)
- net SCK: now also U1.8 (IO15); no longer U1.5 (IO5)
- net VBUS: now also C10.1, U5.3 (VI); no longer R12.1
- net en: now also R13.2
- new net +3V3USB: C11.1, R12.1, U5.2 (VO)
Other:
- moved on the sheet: TP2

Commit message: wow i have a lot to do
Parts:
- removed C11, C3, C4, C6: 1 µF, Capacitor_SMD:C_0603_1608Metric, symbol Device:C
- removed R12: 10 kΩ, Resistor_SMD:R_0402_1005Metric, symbol Device:R
- removed U4, U5: AMS1117-3.3, Package_TO_SOT_SMD:SOT-223-3_TabPin2, symbol Regulator_Linear:AMS1117-3.3
- added D1, D2: PZS52C3V9M1Q, Diode_SMD:D_0402_1005Metric, symbol Diode:BZV55B3V9
- added L1: 1.5uH 70mOhm, Inductor_SMD:L_1008_2520Metric, symbol Device:L
- added R14: 10 kΩ, Resistor_SMD:R_0402_1005Metric, symbol Device:R
- added TP3: VSYS, TestPoint:TestPoint_Keystone_5010-5014_Multipurpose, symbol Connector:TestPoint
- added TP4, TP5, TP6: 3V3, TestPoint:TestPoint_Keystone_5010-5014_Multipurpose, symbol Connector:TestPoint
- added TP7: 3V3, TestPoint:TestPoint_THTPad_D1.0mm_Drill0.5mm, symbol Connector:TestPoint
- added U3: TPS63001, Package_SON:Texas_DRC0010J_ThermalVias, symbol Regulator_Switching:TPS63001
- C10: value 1 µF -> 47 µF
- R10: value 2.4 kΩ -> 13 kΩ
- TP1, TP2: footprint TestPoint:TestPoint_Keystone_5010-5014_Multipurpose -> libraries:smalltestpoint
Connections:
- net +3.3V is gone; now on net +3V3: R13.1, U1.2 (3V3), U2.8 (VCC)
- net +3V3: now also C10.1, D2.1 (K), TP4.1, U3.1 (VOUT), U3.10 (FB)
- net +BATT: no longer R8.1
- net BATTVOLT: now also D1.1 (K)
- net GND: now also U6.4 (/CE), D1.2 (A), D2.2 (A), R14.2, U3.11 (PGND), U3.3 (PGND), U3.9 (GND)
- net MISO: now also TP6.1
- net MOSI: now also TP7.1
- net SCK: now also TP5.1
- net VBUS: no longer C10.1
- net at SW3.1 (A), U6.6 (TS/MR): now also R14.1
- net +4.5V renamed +VSYS
- net +VSYS: now also R8.1, TP3.1, U3.5 (VIN), U3.6 (EN), U3.7 (PS/SYNC), U3.8 (VINA)
- net CHGSWITCH: no longer names the net of U1.38 (IO2)
- net CHGSWITCH: no longer U6.4 (/CE)
- new net: L1.1, U3.2 (L2)
- new net: L1.2, U3.4 (L1)
Other:
- title: (none) -> kiku
- moved on the sheet: R8, R9

Commit message: second attempt of routing
Parts:
- TP3, TP4, TP5, TP6: footprint TestPoint:TestPoint_Keystone_5010-5014_Multipurpose -> libraries:smalltestpoint
- TP7: footprint TestPoint:TestPoint_THTPad_D1.0mm_Drill0.5mm -> libraries:smalltestpoint
Connections:
- net BUSY: now also U1.7 (IO7); no longer U1.5 (IO5)
- net DIO1: now also U1.8 (IO15); no longer U1.9 (IO16)
- net MISO: now also U1.9 (IO16); no longer U1.15 (IO3)
- net MOSI: now also U1.10 (IO17); no longer U1.12 (IO8)
- net RESET: now also U1.12 (IO8); no longer U1.6 (IO6)
- net SCK: now also U1.11 (IO18); no longer U1.8 (IO15)
