File: kiku.kicad_pcb (KiCad board)
At the start: 2 copper layers, 58.8 x 59.6 mm, 35 parts, among them J1 BM02B-SRSS-TB LFSN, J2 USB_C_Receptacle_USB2.0_16P, J3 Conn_Coaxial, SW1 BOOT, SW2 EN, SW3 RESET CHARGER, U1 ESP32-S3-WROOM-1, U2 Wio-sx1262-n, U3 TPS63001, U6 BQ25185DLHR

Commit message: move antenna to other side of board
Parts:
- TP3, TP4, TP5, TP6: footprint TestPoint:TestPoint_Keystone_5010-5014_Multipurpose -> libraries:smalltestpoint
- TP7: footprint TestPoint:TestPoint_THTPad_D1.0mm_Drill0.5mm -> libraries:smalltestpoint
- moved C10 46.1 mm to (166.5, 119.5), turned to 180 degrees
- moved D2 42.3 mm to (166.8, 118.0), turned to 180 degrees
- moved TP3 41.6 mm to (169.2, 120.2)
- moved D1 27.8 mm to (181.6, 75.8), turned to 90 degrees
- moved L1 26.4 mm to (164.4, 122.6), turned to -90 degrees
- moved TP2 22.4 mm to (185.6, 105.2)
- moved TP4 20.9 mm to (169.2, 118.0)
- moved TP1 16.8 mm to (188.4, 105.2)
- moved SW3 9.36 mm to (173.0, 130.2)
- moved R14 9.10 mm to (169.7, 128.8)
- moved U3 6.08 mm to (170.7, 124.5)
- moved R9 3.62 mm to (179.9, 75.8), turned to 90 degrees
- moved R8 2.36 mm to (152.4, 124.6)
- moved C7 0.90 mm to (179.6, 108.8)
- moved C8 0.68 mm to (144.8, 122.6), turned to 90 degrees
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Connections:
- U1 pad 10: unconnected-(U1-IO17-Pad10) -> MOSI
- U1 pad 11: unconnected-(U1-IO18-Pad11) -> SCK
- U1 pad 12: MOSI -> RESET
- U1 pad 15: MISO -> unconnected-(U1-IO3-Pad15)
- U1 pad 5: BUSY -> unconnected-(U1-IO5-Pad5)
- U1 pad 6: RESET -> unconnected-(U1-IO6-Pad6)
- U1 pad 7: unconnected-(U1-IO7-Pad7) -> BUSY
- U1 pad 8: SCK -> DIO1
- U1 pad 9: DIO1 -> MISO
Routing:
- net +3V3: track 0.00 -> 95.5 mm
- net BATTVOLT: track 0.00 -> 72.6 mm, vias 0 -> 2
- net VBUS: track 0.00 -> 51.2 mm, vias 0 -> 2
- net D+: track 0.00 -> 44.9 mm, vias 0 -> 2
- net D-: track 0.00 -> 43.8 mm, vias 0 -> 2
- net MISO: track 0.00 -> 39.9 mm
- net MOSI: track 0.00 -> 37.2 mm
- net SCK: track 0.00 -> 34.4 mm
- net DIO1: track 0.00 -> 34.0 mm
- net BUSY: track 0.00 -> 34.0 mm
- net en: track 0.00 -> 33.0 mm
- net +VSYS: track 0.00 -> 30.5 mm
- net RESET: track 0.00 -> 27.2 mm
- net ANT: track 0.00 -> 20.2 mm
- net +BATT: track 0.00 -> 18.9 mm
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Other:
- board text added: "3V3"
- board text added: "MISO"
- board text added: "MOSI"
- board text added: "SCK"
- board text added: "VSYS"
